Commit message: cleanup

File: kuka_kr210_support/urdf/kr210l150.urdf (robot description, URDF)
Before this commit: robot kuka_kr210, 9 links, 8 joints
Joints:
- removed joint joint_a1
- removed joint joint_a2
- removed joint joint_a3
- removed joint joint_a4
- removed joint joint_a5
- removed joint joint_a6
- added joint joint_1: type revolute, parent base_link, child link_1, origin xyz=-0.00262 0.00097586 0.33099 rpy=0 0 0, axis 0 0 1, limit lower=-3.228859205 upper=3.228859205 effort=0 velocity=2.146755039
- added joint joint_2: type revolute, parent link_1, child link_2, origin xyz=0.35277 -0.037476 0.4192 rpy=0 0 0, axis 0 1 0, limit lower=-0.785398185 upper=1.483529905 effort=0 velocity=2.007128695
- added joint joint_3: type revolute, parent link_2, child link_3, origin xyz=-9.8483E-05 -0.1475 1.2499 rpy=0 0 0, axis 0 1 0, limit lower=-3.66519153 upper=1.134464045 effort=0 velocity=1.954768816
- added joint joint_4: type revolute, parent link_3, child link_4, origin xyz=0.95795 0.184 -0.055059 rpy=0 0 0, axis 1 0 0, limit lower=-6.10865255 upper=6.10865255 effort=0 velocity=3.124139447
- added joint joint_5: type revolute, parent link_4, child link_5, origin xyz=0.542 0 0 rpy=0 0 0, axis 0 1 0, limit lower=-2.181661625 upper=2.181661625 effort=0 velocity=3.001966396
- added joint joint_6: type revolute, parent link_5, child link_6, origin xyz=0.1925 0 0 rpy=0 0 0, axis 1 0 0, limit lower=-6.10865255 upper=6.10865255 effort=0 velocity=3.822271167

File: kuka_kr210_support/urdf/kr210l150_macro.ros2_control.xacro (robot description, xacro)
@@ -15,5 +15,5 @@
         <param name="position_state_following_offset">0.0</param>
       </hardware>
-      <joint name="${prefix}joint_a1">
+      <joint name="${prefix}joint_1">
         <command_interface name="position">     <!-- Add/Remove interfaces as needed -->
           <param name="min">-1</param>
@@ -24,5 +24,5 @@
         </state_interface>
       </joint>
-      <joint name="${prefix}joint_a2">
+      <joint name="${prefix}joint_2">
         <command_interface name="position">     <!-- Add/Remove interfaces as needed -->
           <param name="min">-1</param>
@@ -33,5 +33,5 @@
         </state_interface>
       </joint>
-      <joint name="${prefix}joint_a3">
+      <joint name="${prefix}joint_3">
         <command_interface name="position">     <!-- Add/Remove interfaces as needed -->
           <param name="min">-1</param>
@@ -42,5 +42,5 @@
         </state_interface>
       </joint>
-      <joint name="${prefix}joint_a4">
+      <joint name="${prefix}joint_4">
         <command_interface name="position">     <!-- Add/Remove interfaces as needed -->
           <param name="min">-1</param>
@@ -51,5 +51,5 @@
         </state_interface>
       </joint>
-      <joint name="${prefix}joint_a5">
+      <joint name="${prefix}joint_5">
         <command_interface name="position">     <!-- Add/Remove interfaces as needed -->
           <param name="min">-1</param>
@@ -60,5 +60,5 @@
         </state_interface>
       </joint>
-      <joint name="${prefix}joint_a6">
+      <joint name="${prefix}joint_6">
         <command_interface name="position">     <!-- Add/Remove interfaces as needed -->
           <param name="min">-1</param>

File: kuka_kr210_support/urdf/kr210l150_macro.xacro (robot description, xacro)
@@ -160,5 +160,5 @@
     <link name="${prefix}flange"/>
     <!-- joints -->
-    <joint name="${prefix}joint_a1" type="revolute">
+    <joint name="${prefix}joint_1" type="revolute">
       <origin xyz="-0.00262 0.00097586 0.33099" rpy="0 0 0"/>
       <parent link="${prefix}base_link"/>
@@ -167,5 +167,5 @@
       <limit lower="${radians(-185)}" upper="${radians(185)}" effort="0" velocity="${radians(123)}"/>
     </joint>
-    <joint name="${prefix}joint_a2" type="revolute">
+    <joint name="${prefix}joint_2" type="revolute">
       <origin xyz="0.35277 -0.037476 0.4192" rpy="0 0 0"/>
       <parent link="${prefix}link_1"/>
@@ -174,5 +174,5 @@
       <limit lower="${radians(-45)}" upper="${radians(85)}" effort="0" velocity="${radians(115)}"/>
     </joint>
-    <joint name="${prefix}joint_a3" type="revolute">
+    <joint name="${prefix}joint_3" type="revolute">
       <origin xyz="-9.8483E-05 -0.1475 1.2499" rpy="0 0 0"/>
       <parent link="${prefix}link_2"/>
@@ -181,5 +181,5 @@
       <limit lower="${radians(-210)}" upper="${radians(65)}" effort="0" velocity="${radians(112)}"/>
     </joint>
-    <joint name="${prefix}joint_a4" type="revolute">
+    <joint name="${prefix}joint_4" type="revolute">
       <origin xyz="0.95795 0.184 -0.055059" rpy="0 0 0"/>
       <parent link="${prefix}link_3"/>
@@ -188,5 +188,5 @@
       <limit lower="${radians(-350)}" upper="${radians(350)}" effort="0" velocity="${radians(179)}"/>
     </joint>
-    <joint name="${prefix}joint_a5" type="revolute">
+    <joint name="${prefix}joint_5" type="revolute">
       <origin xyz="0.542 0 0" rpy="0 0 0"/>
       <parent link="${prefix}link_4"/>
@@ -195,5 +195,5 @@
       <limit lower="${radians(-125)}" upper="${radians(125)}" effort="0" velocity="${radians(172)}"/>
     </joint>
-    <joint name="${prefix}joint_a6" type="revolute">
+    <joint name="${prefix}joint_6" type="revolute">
       <origin xyz="0.1925 0 0" rpy="0 0 0"/>
       <parent link="${prefix}link_5"/>

File: kuka_kr210_support/urdf/kr210r2700_.urdf (robot description, URDF)
Before this commit: robot kuka_kr210, 9 links, 8 joints
Joints:
- removed joint joint_a1
- removed joint joint_a2
- removed joint joint_a3
- removed joint joint_a4
- removed joint joint_a5
- removed joint joint_a6
- added joint joint_1: type revolute, parent base_link, child link_1, origin xyz=-0.00262 0.00097586 0.33099 rpy=0 0 0, axis 0 0 1, limit lower=-3.228859205 upper=3.228859205 effort=0 velocity=2.146755039
- added joint joint_2: type revolute, parent link_1, child link_2, origin xyz=0.35277 -0.037476 0.4192 rpy=0 0 0, axis 0 1 0, limit lower=-0.785398185 upper=1.483529905 effort=0 velocity=2.007128695
- added joint joint_3: type revolute, parent link_2, child link_3, origin xyz=-9.8483E-05 -0.1475 1.2499 rpy=0 0 0, axis 0 1 0, limit lower=-3.66519153 upper=1.134464045 effort=0 velocity=1.954768816
- added joint joint_4: type revolute, parent link_3, child link_4, origin xyz=0.95795 0.184 -0.055059 rpy=0 0 0, axis 1 0 0, limit lower=-6.10865255 upper=6.10865255 effort=0 velocity=3.124139447
- added joint joint_5: type revolute, parent link_4, child link_5, origin xyz=0.542 0 0 rpy=0 0 0, axis 0 1 0, limit lower=-2.181661625 upper=2.181661625 effort=0 velocity=3.001966396
- added joint joint_6: type revolute, parent link_5, child link_6, origin xyz=0.1925 0 0 rpy=0 0 0, axis 1 0 0, limit lower=-6.10865255 upper=6.10865255 effort=0 velocity=3.822271167

File: kuka_kr210_support/urdf/kr210r2700_macro.ros2_control.xacro (robot description, xacro)
@@ -15,5 +15,5 @@
         <param name="position_state_following_offset">0.0</param>
       </hardware>
-      <joint name="${prefix}joint_a1">
+      <joint name="${prefix}joint_1">
         <command_interface name="position">     <!-- Add/Remove interfaces as needed -->
           <param name="min">-1</param>
@@ -24,5 +24,5 @@
         </state_interface>
       </joint>
-      <joint name="${prefix}joint_a2">
+      <joint name="${prefix}joint_2">
         <command_interface name="position">     <!-- Add/Remove interfaces as needed -->
           <param name="min">-1</param>
@@ -33,5 +33,5 @@
         </state_interface>
       </joint>
-      <joint name="${prefix}joint_a3">
+      <joint name="${prefix}joint_3">
         <command_interface name="position">     <!-- Add/Remove interfaces as needed -->
           <param name="min">-1</param>
@@ -42,5 +42,5 @@
         </state_interface>
       </joint>
-      <joint name="${prefix}joint_a4">
+      <joint name="${prefix}joint_4">
         <command_interface name="position">     <!-- Add/Remove interfaces as needed -->
           <param name="min">-1</param>
@@ -51,5 +51,5 @@
         </state_interface>
       </joint>
-      <joint name="${prefix}joint_a5">
+      <joint name="${prefix}joint_5">
         <command_interface name="position">     <!-- Add/Remove interfaces as needed -->
           <param name="min">-1</param>
@@ -60,5 +60,5 @@
         </state_interface>
       </joint>
-      <joint name="${prefix}joint_a6">
+      <joint name="${prefix}joint_6">
         <command_interface name="position">     <!-- Add/Remove interfaces as needed -->
           <param name="min">-1</param>

File: kuka_kr210_support/urdf/kr210r2700_macro.xacro (robot description, xacro)
@@ -160,5 +160,5 @@
     <link name="${prefix}tool0"/>
     <!-- joints -->
-    <joint name="${prefix}joint_a1" type="revolute">
+    <joint name="${prefix}joint_1" type="revolute">
       <origin xyz="0 0 0.240" rpy="0 0 0"/>
       <parent link="${prefix}base_link"/>
@@ -167,5 +167,5 @@
       <limit lower="${radians(-185)}" upper="${radians(185)}" effort="0" velocity="${radians(123)}"/>
     </joint>
-    <joint name="${prefix}joint_a2" type="revolute">
+    <joint name="${prefix}joint_2" type="revolute">
       <origin xyz="0.330 0 0.405" rpy="0 ${radians(90)} 0"/>
       <parent link="${prefix}link_1"/>
@@ -174,5 +174,5 @@
       <limit lower="${radians(-140)}" upper="${radians(-5)}" effort="0" velocity="${radians(115)}"/>
     </joint>
-    <joint name="${prefix}joint_a3" type="revolute">
+    <joint name="${prefix}joint_3" type="revolute">
       <origin xyz="0 0 1.15" rpy="0 0 0"/>
       <parent link="${prefix}link_2"/>
@@ -181,5 +181,5 @@
       <limit lower="${radians(-120)}" upper="${radians(168)}" effort="0" velocity="${radians(112)}"/>
     </joint>
-    <joint name="${prefix}joint_a4" type="revolute">
+    <joint name="${prefix}joint_4" type="revolute">
       <origin xyz="-0.115 0 1.22" rpy="0 0 0"/>
       <parent link="${prefix}link_3"/>
@@ -188,5 +188,5 @@
       <limit lower="${radians(-350)}" upper="${radians(350)}" effort="0" velocity="${radians(179)}"/>
     </joint>
-    <joint name="${prefix}joint_a5" type="revolute">
+    <joint name="${prefix}joint_5" type="revolute">
       <origin xyz="0 0 0" rpy="${radians(-90)} 0 0"/>
       <parent link="${prefix}link_4"/>
@@ -195,5 +195,5 @@
       <limit lower="${radians(-125)}" upper="${radians(125)}" effort="0" velocity="${radians(172)}"/>
     </joint>
-    <joint name="${prefix}joint_a6" type="revolute">
+    <joint name="${prefix}joint_6" type="revolute">
       <origin xyz="0 -0.215 0" rpy="${radians(90)} 0 0"/>
       <parent link="${prefix}link_5"/>

File: kuka_resources/urdf/common_macro.ros2_control.xacro (robot description, xacro)
@@ -8,5 +8,5 @@
         </xacro:if>
       </hardware>
-      <joint name="${prefix}joint_a1">
+      <joint name="${prefix}joint_1">
         <command_interface name="position">
           <param name="min">-1</param>
@@ -17,5 +17,5 @@
         </state_interface>
       </joint>
-      <joint name="${prefix}joint_a2">
+      <joint name="${prefix}joint_2">
         <command_interface name="position">
           <param name="min">-1</param>
@@ -26,5 +26,5 @@
         </state_interface>
 	  </joint>
-      <joint name="${prefix}joint_a3">
+      <joint name="${prefix}joint_3">
         <command_interface name="position">
           <param name="min">-1</param>
@@ -35,5 +35,5 @@
         </state_interface>
 	  </joint>
-      <joint name="${prefix}joint_a4">
+      <joint name="${prefix}joint_4">
         <command_interface name="position">
           <param name="min">-1</param>
@@ -44,5 +44,5 @@
         </state_interface>
       </joint>
-      <joint name="${prefix}joint_a5">
+      <joint name="${prefix}joint_5">
         <command_interface name="position">
           <param name="min">-1</param>
@@ -53,5 +53,5 @@
         </state_interface>
       </joint>
-      <joint name="${prefix}joint_a6">
+      <joint name="${prefix}joint_6">
         <command_interface name="position">
           <param name="min">-1</param>
