Commit message: update tool0

File: kuka_kr210_support/urdf/kr210r2700_macro.xacro (robot description, xacro)
@@ -205,5 +205,5 @@
       <parent link="${prefix}link_6"/>
       <child link="${prefix}tool0"/>
-      <origin xyz="0 0 0" rpy="0 0 0"/>
+      <origin xyz="0 0 0.008" rpy="0 0 0"/>
     </joint>
     <!-- ROS base_link to KUKA $ROBROOT coordinate system transform -->

Commit message: Restrict joint 3

File: kuka_kr210_support/urdf/kr210r2700_macro.xacro (robot description, xacro)
@@ -179,5 +179,5 @@
       <child link="${prefix}link_3"/>
       <axis xyz="0 1 0"/>
-      <limit lower="${radians(-120)}" upper="${radians(168)}" effort="0" velocity="${radians(112)}"/>
+      <limit lower="${radians(55)}" upper="${radians(168)}" effort="0" velocity="${radians(112)}"/>
     </joint>
     <joint name="${prefix}joint_4" type="revolute">

Commit message: change r2700 limits

File: kuka_kr210_support/urdf/kr210r2700_macro.xacro (robot description, xacro)
@@ -179,5 +179,5 @@
       <child link="${prefix}link_3"/>
       <axis xyz="0 1 0"/>
-      <limit lower="${radians(55)}" upper="${radians(168)}" effort="0" velocity="${radians(112)}"/>
+      <limit lower="${radians(0)}" upper="${radians(168)}" effort="0" velocity="${radians(112)}"/>
     </joint>
     <joint name="${prefix}joint_4" type="revolute">

Commit message: checkpoint

File: kuka_kr210_support/urdf/kr210r2700_macro.xacro (robot description, xacro)
@@ -142,5 +142,5 @@
       </inertial>
       <visual>
-        <origin xyz="0 0 0" rpy="0 0 0"/>
+        <origin xyz="0 0 0" rpy="0 0 -1.92"/>
         <geometry>
           <mesh filename="file://$(find kuka_kr210_support)/meshes/kr210r2700/visual/link_6.stl"/>
@@ -151,5 +151,5 @@
       </visual>
       <collision>
-        <origin xyz="0 0 0" rpy="0 0 0"/>
+        <origin xyz="0 0 0" rpy="0 0 -0.785398"/>
         <geometry>
           <mesh filename="file://$(find kuka_kr210_support)/meshes/kr210r2700/collision/link_6.stl"/>

Commit message: fix: remove 8mm offset

File: kuka_kr210_support/urdf/kr210r2700_macro.xacro (robot description, xacro)
@@ -205,5 +205,5 @@
       <parent link="${prefix}link_6"/>
       <child link="${prefix}tool0"/>
-      <origin xyz="0 0 0.008" rpy="0 0 0"/>
+      <origin xyz="0 0 0.0" rpy="0 0 0"/>
     </joint>
     <!-- ROS base_link to KUKA $ROBROOT coordinate system transform -->
